File: rev1.c/OLED_1.5_128X128_breakout.kicad_pcb (KiCad board)
At the start: 2 copper layers, 44 x 44 mm, 20 parts, among them P1 BREAKOUT, U1 FAN5331SX, U2 ER_OLED015_1C

Commit message: finished routing rev 1.c
Parts:
- moved C6 9.81 mm to (60.5, 69.7)
- moved C3 6.50 mm to (60.5, 62.5), turned to 180 degrees
- moved D3 2.78 mm to (67.4, 68.7)
- moved R4 2.73 mm to (67.4, 64.1)
- moved C5 2.64 mm to (60.5, 66.1), turned to 180 degrees
- moved D2 2.12 mm to (65.0, 68.7)
- moved C7 2.01 mm to (65.0, 64.1)
Connections:
- P1 pad 11: /D1/SDIN -> /E/RD#
- P1 pad 12: /D2 -> /R/W#
- P1 pad 13: /D3 -> /BS0
- P1 pad 14: /D4 -> /BS1
- P1 pad 15: /D5 -> /CS#
- P1 pad 16: /D6 -> /D/C#
- P1 pad 17: /D7 -> /RES#
- P1 pad 3: /RES# -> /D7
- P1 pad 4: /D/C# -> /D6
- P1 pad 5: /CS# -> /D5
- P1 pad 6: /BS1 -> /D4
- P1 pad 7: /BS0 -> /D3
- P1 pad 8: /R/W# -> /D2
- P1 pad 9: /E/RD# -> /D1/SDIN
Routing:
- net /RES#: track 0.00 -> 36.9 mm
- net /E/RD#: track 0.22 -> 36.9 mm, vias 0 -> 4
- net /D7: track 0.00 -> 35.9 mm
- net /D/C#: track 0.00 -> 35.8 mm
- net /CS#: track 0.00 -> 35.2 mm
- net /BS1: track 0.00 -> 34.1 mm
- net /D0/SCK: track 0.00 -> 33.9 mm, vias 0 -> 2
- net /D6: track 0.00 -> 33.8 mm
- net /BS0: track 0.00 -> 33.2 mm
- net /D5: track 0.28 -> 32.9 mm
- net /R/W#: track 0.00 -> 32.4 mm
- net /D4: track 0.00 -> 32.0 mm
- net /D3: track 0.00 -> 31.2 mm
- net /D2: track 0.00 -> 30.3 mm
- net /D1/SDIN: track 0.00 -> 30.1 mm
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