File: rev1.c/OLED_1.5_128X128_breakout.sch (KiCad schematic (older format))
At the start: 18 parts, among them P1 BREAKOUT, U1 FAN5331SX, U2 ER_OLED015_1C

Commit message: finished routing rev 1.c
Connections:
- net BS0: now also P1.13 (P13); no longer P1.7 (P7)
- net BS1: now also P1.14 (P14); no longer P1.6 (P6)
- net CS#: now also P1.15 (P15); no longer P1.5 (P5)
- net D/C#: now also P1.16 (P16); no longer P1.4 (P4)
- net D1/SDIN: now also P1.9 (P9); no longer P1.11 (P11)
- net D2: now also P1.8 (P8); no longer P1.12 (P12)
- net D3: now also P1.7 (P7); no longer P1.13 (P13)
- net D4: now also P1.6 (P6); no longer P1.14 (P14)
- net D5: now also P1.5 (P5); no longer P1.15 (P15)
- net D6: now also P1.4 (P4); no longer P1.16 (P16)
- net D7: now also P1.3 (P3); no longer P1.17 (P17)
- net E/RD#: now also P1.11 (P11); no longer P1.9 (P9)
- net R/W#: now also P1.12 (P12); no longer P1.8 (P8)
- net RES#: now also P1.17 (P17); no longer P1.3 (P3)
Changed lines of the file:
@@
 RES#
 Wire Wire Line
-	4025 1575 3625 1575
-Text Label 3625 1575 0    60   ~ 0
+	4025 2975 3625 2975
+Text Label 3625 2975 0    60   ~ 0
 D7
 Wire Wire Line
-	4025 1675 3625 1675
-Text Label 3625 1675 0    60   ~ 0
+	4025 2875 3625 2875
+Text Label 3625 2875 0    60   ~ 0
 D6
 Wire Wire Line
-	4025 1775 3625 1775
-Text Label 3625 1775 0    60   ~ 0
+	4025 2775 3625 2775
+Text Label 3625 2775 0    60   ~ 0
 D5
 Wire Wire Line
-	4025 1875 3625 1875
-Text Label 3625 1875 0    60   ~ 0
+	4025 2675 3625 2675
+Text Label 3625 2675 0    60   ~ 0
 D4
 Wire Wire Line
-	4025 1975 3625 1975
-Text Label 3625 1975 0    60   ~ 0
+	4025 2575 3625 2575
+Text Label 3625 2575 0    60   ~ 0
 D3
 Wire Wire Line
-	4025 2075 3625 2075
-Text Label 3625 2075 0    60   ~ 0
+	4025 2475 3625 2475
+Text Label 3625 2475 0    60   ~ 0
 D2
 Wire Wire Line
-	4025 2175 3625 2175
-Text Label 3625 2175 0    60   ~ 0
+	4025 2375 3625 2375
+Text Label 3625 2375 0    60   ~ 0
 D1/SDIN
 Wire Wire Line
@@
 D0/SCK
 Wire Wire Line
-	4025 2375 3625 2375
-Text Label 3625 2375 0    60   ~ 0
+	4025 2175 3625 2175
+Text Label 3625 2175 0    60   ~ 0
 E/RD#
 Wire Wire Line
-	4025 2475 3625 2475
-Text Label 3625 2475 0    60   ~ 0
+	4025 2075 3625 2075
+Text Label 3625 2075 0    60   ~ 0
 R/W#
 Wire Wire Line
-	4025 2575 3625 2575
-Text Label 3625 2575 0    60   ~ 0
+	4025 1975 3625 1975
+Text Label 3625 1975 0    60   ~ 0
 BS0
 Wire Wire Line
-	4025 2675 3625 2675
-Text Label 3625 2675 0    60   ~ 0
+	4025 1875 3625 1875
+Text Label 3625 1875 0    60   ~ 0
 BS1
 Wire Wire Line
-	4025 2775 3625 2775
-Text Label 3625 2775 0    60   ~ 0
+	4025 1775 3625 1775
+Text Label 3625 1775 0    60   ~ 0
 CS#
 Wire Wire Line
-	4025 2875 3625 2875
-Text Label 3625 2875 0    60   ~ 0
+	4025 1675 3625 1675
+Text Label 3625 1675 0    60   ~ 0
 D/C#
 Wire Wire Line
-	4025 2975 3625 2975
-Text Label 3625 2975 0    60   ~ 0
+	4025 1575 3625 1575
+Text Label 3625 1575 0    60   ~ 0
 RES#
 Wire Wire Line
